Commit message: reconfigured the launch package to another package with urdf description

File: src/ros2_ws/src/morve_description/description/urdf/morve_description.urdf.xacro (robot description, xacro)
@@ -41,4 +41,19 @@
         </visual>
     </link>
+    <!-- Test of inserting mesh of sonar holder to urdf -->
+    <joint name="${prefix}front_sonar_holder_joint" type="fixed">
+        <parent link="${prefix}base_link"/>
+        <child link="${prefix}front_sonar_holder"/>
+        <origin xyz="0.0 ${-base_length/2} ${z_offset}" rpy="0.0 0.0 0.0"/>
+    </joint>
+    <link name="${prefix}front_sonar_holder">
+        <visual>
+            <origin xyz="-0.025 0.0 0.0" rpy="0.0 0.0 0.0"/>
+            <geometry>
+                <mesh filename="package://morve_description/description/meshes/HC_SR04_2021_holder.stl" scale="0.001 0.001 0.001"/>
+            </geometry>
+            <material name="blue"/>
+        </visual>
+    </link>
     </xacro:macro>
 </robot>

Commit message: created more macros for urdf file and added meshes for robot representation

File: src/ros2_ws/src/morve_description/description/urdf/morve_description.urdf.xacro (robot description, xacro)
@@ -1,59 +1,89 @@
 <?xml version="1.0"?>
 <robot xmlns:xacro="http://www.ros.org/wiki/xacro">
+    <!-- Macro with constants  -->
+    <xacro:macro name="morve_constants">
+        <xacro:property name="PI" value="3.1415926535897931" scope="parent" />
+        <xacro:property name="base_mass" value="0.3" scope="parent" /> <!-- arbitrary value for base mass -->
+        <xacro:property name="base_width" value="0.16" scope="parent" />
+        <xacro:property name="base_length" value="0.2" scope="parent" />
+        <xacro:property name="base_height" value="0.005" scope="parent" />
+        <xacro:property name="wheel_mass" value="0.3" scope="parent" /> <!-- arbitrary value for wheel mass -->
+        <xacro:property name="track_width" value="0.2" scope="parent" />
+        <xacro:property name="wheel_base" value="0.12" scope="parent" />
+        <xacro:property name="track_width_half" value="${track_width/2}" scope="parent" />
+        <xacro:property name="wheel_base_half" value="${wheel_base/2}" scope="parent" />
+        <xacro:property name="z_offset" value="${base_height/2}" scope="parent" />
+        <xacro:property name="mesh_scale" value="0.001 0.001 0.001" scope="parent" />
+        <xacro:property name="wheel_length" value="0.025" scope="parent" />
+        <xacro:property name="wheel_radius" value="0.0325" scope="parent" />
+    </xacro:macro>
+    <!-- Macro for Sonar holder -->
+    <xacro:macro name="sonar_holder" params="name prefix parent_link joint_x joint_y joint_z joint_yaw">
+        <!-- Include constants -->
+        <xacro:morve_constants />
+        <joint name="${prefix}${name}_joint" type="fixed">
+            <parent link="${prefix}${parent_link}"/>
+            <child link="${prefix}${name}"/>
+            <origin xyz="${joint_x} ${joint_y} ${joint_z}" rpy="0.0 0.0 ${joint_yaw}"/>
+        </joint>
+        <link name="${prefix}${name}">
+            <visual>
+                <origin xyz="-0.025 0.0 0.0" rpy="0.0 0.0 0.0"/>
+                <geometry>
+                    <mesh filename="package://morve_description/description/meshes/sonar_holder.stl" scale="${mesh_scale}"/>
+                </geometry>
+                <material name="blue"/>
+            </visual>
+        </link>
+    </xacro:macro>
+    <!-- Macro for wheel -->
+    <xacro:macro name="robotic_wheel" params="name prefix parent_link joint_x joint_y joint_z">
+        <!-- Include constants -->
+        <xacro:morve_constants />
+        <joint name="${name}_joint" type="continuous">
+            <parent link="${prefix}${parent_link}"/>
+            <child link="${prefix}${name}"/>
+            <axis xyz="0 0 1"/>
+            <origin xyz="${joint_x} ${joint_y} ${joint_z}" rpy="0 ${PI/2} 0"/>
+        </joint>
+        <link name="${prefix}${name}">
+            <visual>
+                <geometry>
+                    <cylinder radius="${wheel_radius}" length="${wheel_length}"/>
+                </geometry>
+                <material name="green"/>
+            </visual>
+        </link>
+    </xacro:macro>
+    <!-- Macro for whole robot -->
     <xacro:macro name="morve_description_urdf" params="prefix">
-    <!-- Constants for robot dimensions -->
-    <xacro:property name="PI" value="3.1415926535897931"/>
-    <xacro:property name="base_mass" value="0.3" /> <!-- arbitrary value for base mass -->
-    <xacro:property name="base_width" value="0.16" />
-    <xacro:property name="base_length" value="0.2" />
-    <xacro:property name="base_height" value="0.005" />
-    <xacro:property name="wheel_mass" value="0.3" /> <!-- arbitrary value for wheel mass -->
-    <xacro:property name="wheel_length" value="0.025" />
-    <xacro:property name="wheel_radius" value="0.0325" />
-    <xacro:property name="track_width" value="0.2" />
-    <xacro:property name="wheel_base" value="0.12" />
-    <xacro:property name="track_width_half" value="${track_width/2}"/>
-    <xacro:property name="wheel_base_half" value="${wheel_base/2}" />
-    <xacro:property name="z_offset" value="${base_height/2}" /> <!-- Space btw top of beam and the each joint -->
-    <!-- Base link -->
-    <link name="${prefix}base_link">
-        <visual>
-             <origin xyz="0.0 0.0 0.0" rpy="0.0 0.0 0.0"/>
-             <geometry>
-                <box size="${base_width} ${base_length} ${base_height}"/>
-             </geometry>
-             <material name="white"/>
-        </visual>
-    </link>
-    <!-- Front left wheel joint and link (part) -->
-    <joint name="${prefix}front_left_wheel_joint" type="continuous">
-        <parent link="${prefix}base_link"/>
-        <child link="${prefix}front_left_wheel"/>
-        <axis xyz="0 0 1"/>
-        <origin xyz="${track_width_half} ${-wheel_base_half} ${z_offset}" rpy="0 ${PI/2} 0"/>
-    </joint>
-    <link name="${prefix}front_left_wheel">
-        <visual>
-            <geometry>
-                <cylinder radius="${wheel_radius}" length="${wheel_length}"/>
-            </geometry>
-            <material name="green"/>
-        </visual>
-    </link>
-    <!-- Test of inserting mesh of sonar holder to urdf -->
-    <joint name="${prefix}front_sonar_holder_joint" type="fixed">
-        <parent link="${prefix}base_link"/>
-        <child link="${prefix}front_sonar_holder"/>
-        <origin xyz="0.0 ${-base_length/2} ${z_offset}" rpy="0.0 0.0 0.0"/>
-    </joint>
-    <link name="${prefix}front_sonar_holder">
-        <visual>
-            <origin xyz="-0.025 0.0 0.0" rpy="0.0 0.0 0.0"/>
-            <geometry>
-                <mesh filename="package://morve_description/description/meshes/HC_SR04_2021_holder.stl" scale="0.001 0.001 0.001"/>
-            </geometry>
-            <material name="blue"/>
-        </visual>
-    </link>
+        <!-- Include constants -->
+        <xacro:morve_constants />
+        <!-- Base link -->
+        <link name="${prefix}base_link">
+            <visual>
+                <origin xyz="${base_width/2} ${-base_length/2} ${-z_offset}" rpy="0.0 0.0 ${PI/2}"/>
+                <geometry>
+                    <mesh filename="package://morve_description/description/meshes/base_plate_with_holes.stl" scale="${mesh_scale}"/>
+                </geometry>
+                <material name="white"/>
+            </visual>
+        </link>
+        <!-- Instantiation of robotic wheels -->
+        <xacro:robotic_wheel name="front_left_wheel" prefix="${prefix}" parent_link="base_link"
+                            joint_x="${track_width_half}" joint_y="${-wheel_base_half}" joint_z="${z_offset}"/>
+        <xacro:robotic_wheel name="rear_left_wheel" prefix="${prefix}" parent_link="base_link"
+                            joint_x="${track_width_half}" joint_y="${wheel_base_half}" joint_z="${z_offset}"/>
+        <xacro:robotic_wheel name="front_right_wheel" prefix="${prefix}" parent_link="base_link"
+                            joint_x="${-track_width_half}" joint_y="${-wheel_base_half}" joint_z="${z_offset}"/>
+        <xacro:robotic_wheel name="rear_right_wheel" prefix="${prefix}" parent_link="base_link"
+                            joint_x="${-track_width_half}" joint_y="${wheel_base_half}" joint_z="${z_offset}"/>
+        <!-- Instantiation of sonar holders -->
+        <xacro:sonar_holder name="front_sonar_holder" prefix="${prefix}" parent_link="base_link"
+                            joint_x="0.0" joint_y="${-base_length/2}" joint_z="${z_offset}" joint_yaw="0.0"/>
+        <xacro:sonar_holder name="left_side_sonar_holder" prefix="${prefix}" parent_link="base_link"
+                            joint_x="${base_width/2}" joint_y="0.0" joint_z="${z_offset}" joint_yaw="${PI/2}"/>
+        <xacro:sonar_holder name="right_side_sonar_holder" prefix="${prefix}" parent_link="base_link"
+                            joint_x="${-base_width/2}" joint_y="0.0" joint_z="${z_offset}" joint_yaw="${-PI/2}"/>
     </xacro:macro>
 </robot>

Commit message: refined macros inside of morve_description.urdf.xacro

File: src/ros2_ws/src/morve_description/description/urdf/morve_description.urdf.xacro (robot description, xacro)
@@ -19,13 +19,13 @@
     </xacro:macro>
     <!-- Macro for Sonar holder -->
-    <xacro:macro name="sonar_holder" params="name prefix parent_link joint_x joint_y joint_z joint_yaw">
+    <xacro:macro name="sonar_holder" params="prefix parent_link joint_x joint_y joint_z joint_yaw">
         <!-- Include constants -->
         <xacro:morve_constants />
-        <joint name="${prefix}${name}_joint" type="fixed">
-            <parent link="${prefix}${parent_link}"/>
-            <child link="${prefix}${name}"/>
+        <joint name="${prefix}_sonar_holder_joint" type="fixed">
+            <parent link="${parent_link}"/>
+            <child link="${prefix}_sonar_holder"/>
             <origin xyz="${joint_x} ${joint_y} ${joint_z}" rpy="0.0 0.0 ${joint_yaw}"/>
         </joint>
-        <link name="${prefix}${name}">
+        <link name="${prefix}_sonar_holder">
             <visual>
                 <origin xyz="-0.025 0.0 0.0" rpy="0.0 0.0 0.0"/>
@@ -38,14 +38,14 @@
     </xacro:macro>
     <!-- Macro for wheel -->
-    <xacro:macro name="robotic_wheel" params="name prefix parent_link joint_x joint_y joint_z">
+    <xacro:macro name="robotic_wheel" params="prefix parent_link rear left">
         <!-- Include constants -->
         <xacro:morve_constants />
-        <joint name="${name}_joint" type="continuous">
-            <parent link="${prefix}${parent_link}"/>
-            <child link="${prefix}${name}"/>
+        <joint name="${prefix}_wheel_joint" type="continuous">
+            <parent link="${parent_link}"/>
+            <child link="${prefix}_wheel"/>
             <axis xyz="0 0 1"/>
-            <origin xyz="${joint_x} ${joint_y} ${joint_z}" rpy="0 ${PI/2} 0"/>
+            <origin xyz="${left*track_width_half} ${rear*wheel_base_half} ${z_offset}" rpy="0 ${PI/2} 0"/>
         </joint>
-        <link name="${prefix}${name}">
+        <link name="${prefix}_wheel">
             <visual>
                 <geometry>
@@ -71,18 +71,18 @@
         </link>
         <!-- Instantiation of robotic wheels -->
-        <xacro:robotic_wheel name="front_left_wheel" prefix="${prefix}" parent_link="base_link"
-                            joint_x="${track_width_half}" joint_y="${-wheel_base_half}" joint_z="${z_offset}"/>
-        <xacro:robotic_wheel name="rear_left_wheel" prefix="${prefix}" parent_link="base_link"
-                            joint_x="${track_width_half}" joint_y="${wheel_base_half}" joint_z="${z_offset}"/>
-        <xacro:robotic_wheel name="front_right_wheel" prefix="${prefix}" parent_link="base_link"
-                            joint_x="${-track_width_half}" joint_y="${-wheel_base_half}" joint_z="${z_offset}"/>
-        <xacro:robotic_wheel name="rear_right_wheel" prefix="${prefix}" parent_link="base_link"
-                            joint_x="${-track_width_half}" joint_y="${wheel_base_half}" joint_z="${z_offset}"/>
+        <xacro:robotic_wheel prefix="${prefix}front_left" parent_link="${prefix}base_link"
+                             rear="-1" left="1" />
+        <xacro:robotic_wheel prefix="${prefix}rear_left" parent_link="${prefix}base_link"
+                             rear="1" left="1" />
+        <xacro:robotic_wheel prefix="${prefix}front_right" parent_link="${prefix}base_link"
+                             rear="-1" left="-1" />
+        <xacro:robotic_wheel prefix="${prefix}rear_right" parent_link="${prefix}base_link"
+                             rear="1" left="-1" />
         <!-- Instantiation of sonar holders -->
-        <xacro:sonar_holder name="front_sonar_holder" prefix="${prefix}" parent_link="base_link"
+        <xacro:sonar_holder prefix="${prefix}front" parent_link="${prefix}base_link"
                             joint_x="0.0" joint_y="${-base_length/2}" joint_z="${z_offset}" joint_yaw="0.0"/>
-        <xacro:sonar_holder name="left_side_sonar_holder" prefix="${prefix}" parent_link="base_link"
+        <xacro:sonar_holder prefix="${prefix}left_side" parent_link="${prefix}base_link"
                             joint_x="${base_width/2}" joint_y="0.0" joint_z="${z_offset}" joint_yaw="${PI/2}"/>
-        <xacro:sonar_holder name="right_side_sonar_holder" prefix="${prefix}" parent_link="base_link"
+        <xacro:sonar_holder prefix="${prefix}right_side" parent_link="${prefix}base_link"
                             joint_x="${-base_width/2}" joint_y="0.0" joint_z="${z_offset}" joint_yaw="${-PI/2}"/>
     </xacro:macro>
