Commit message: finally got the hardware interface motor_interface running

File: src/ros2_ws/src/morve_description/description/urdf/ros2_control/morve.ros2_control.xacro (robot description, xacro)
@@ -7,5 +7,5 @@
         <param name="motor_hat_i2c_addr">0x60</param>
       </hardware>
-      <joint name="${prefix}front_left_motor">
+      <joint name="${prefix}front_left_wheel_joint">
         <param name="motor_hat_output_mapping">motor0</param>
         <param name="encoder_line_A_gpio_pin">gpio7</param>

Commit message: rewrote the hardware interface component for the wheels with encoder and modified configurations

File: src/ros2_ws/src/morve_description/description/urdf/ros2_control/morve.ros2_control.xacro (robot description, xacro)
@@ -19,9 +19,10 @@
         <state_interface name="velocity"/>
       </joint>
-      <!--
-      <joint name="${prefix}rear_left_motor">
-        <param name="motor_hat_output_mapping">motor2</param>
+      <joint name="${prefix}rear_left_wheel_joint">
+        <param name="motor_hat_output_mapping">motor1</param>
         <param name="encoder_line_A_gpio_pin">gpio6</param>
         <param name="encoder_line_B_gpio_pin">gpio12</param>
+        <param name="encoder_pulses_per_rotation">265</param>
+        <param name="wheel_diameter_metres">0.065</param>
         <command_interface name="effort">
           <param name="min">-1024</param>
@@ -30,8 +31,10 @@
         <state_interface name="velocity"/>
       </joint>
-      <joint name="${prefix}front_right_motor">
-        <param name="motor_hat_output_mapping">motor3</param>
+      <joint name="${prefix}front_right_wheel_joint">
+        <param name="motor_hat_output_mapping">motor2</param>
         <param name="encoder_line_A_gpio_pin">gpio16</param>
         <param name="encoder_line_B_gpio_pin">gpio13</param>
+        <param name="encoder_pulses_per_rotation">265</param>
+        <param name="wheel_diameter_metres">0.065</param>
         <command_interface name="effort">
           <param name="min">-1024</param>
@@ -40,8 +43,10 @@
         <state_interface name="velocity"/>
       </joint>
-      <joint name="${prefix}rear_right_motor">
-        <param name="motor_hat_output_mapping">motor4</param>
+      <joint name="${prefix}rear_right_wheel_joint">
+        <param name="motor_hat_output_mapping">motor3</param>
         <param name="encoder_line_A_gpio_pin">gpio20</param>
         <param name="encoder_line_B_gpio_pin">gpio19</param>
+        <param name="encoder_pulses_per_rotation">265</param>
+        <param name="wheel_diameter_metres">0.065</param>
         <command_interface name="effort">
           <param name="min">-1024</param>
@@ -50,5 +55,4 @@
         <state_interface name="velocity"/>
       </joint>
-      -->
     </ros2_control>
   </xacro:macro>
